Commit message: add velocity control

File: robot_golf/env/data/kuka_iiwa/model_0.urdf (robot description, URDF)
Before this commit: robot lbr_iiwa, 9 links, 8 joints
Links:
- added link base_link_0
- added link world_link
Joints:
- added joint x: type prismatic, parent world_link, child base_link_0, axis 1 0 0, limit lower=-2 upper=2 velocity=0
- added joint y: type prismatic, parent base_link_0, child lbr_iiwa_link_0, axis 0 1 0, limit lower=-2 upper=2 velocity=1.0
- joint lbr_iiwa_joint_7: type revolute -> fixed

Commit message: add pipeline

File: robot_golf/env/data/kuka_iiwa/model_0.urdf (robot description, URDF)
Before this commit: robot lbr_iiwa, 11 links, 10 joints
Joints:
- joint x: limit lower=-2 upper=2 velocity=0 -> lower=-5 upper=2 velocity=1.0
